File: Navi-KiCAD/GPS.sch (KiCad schematic (older format))
At the start: 6 parts, among them J6 0734120110, U9 MAX-M8W-0

Commit message: Completed key routing.
Parts:
- renumbered C22 to C80, C23 to C81, C53 to C82, J6 to J3, R14 to R36
Changed lines of the file:
@@
 $EndDescr
 $Comp
-L CONN_COAXIAL J6
+L CONN_COAXIAL J3
 U 1 1 58AF1B18
 P 6750 3450
-F 0 "J6" H 6850 3426 50  0000 L CNN
+F 0 "J3" H 6850 3426 50  0000 L CNN
 F 1 "0734120110" H 6850 3335 50  0000 L CNN
 F 2 "Connectors_Molex:Molex_Microcoaxial_RF" H -350 750 50  0001 C CNN
@@
 RF_GPS_ANT
 $Comp
-L R R14
+L R R36
 U 1 1 58B486B6
 P 5150 2600
-F 0 "R14" V 5050 2500 50  0000 C CNN
+F 0 "R36" V 5050 2500 50  0000 C CNN
 F 1 "ERJ-14YJ100U" V 5250 2600 50  0000 C CNN
 F 2 "Resistors_SMD:R_1210" V -1600 -100 50  0001 C CNN
@@
 	5600 3150 5250 3150
 $Comp
-L C C53
+L C C82
 U 1 1 58B48916
 P 5900 2850
-F 0 "C53" H 6015 3002 50  0000 L CNN
+F 0 "C82" H 6015 3002 50  0000 L CNN
 F 1 "0.01u" H 6015 2911 50  0000 L CNN
 F 2 "Capacitors_SMD:C_0402" H 188 0   50  0001 C CNN
@@
 $EndComp
 $Comp
-L C C23
+L C C81
 U 1 1 58B4A12C
 P 4150 2350
-F 0 "C23" H 4265 2502 50  0000 L CNN
+F 0 "C81" H 4265 2502 50  0000 L CNN
 F 1 "0.01u" H 4265 2411 50  0000 L CNN
 F 2 "Capacitors_SMD:C_0402" H -1562 -500 50  0001 C CNN
@@
 $EndComp
 $Comp
-L C C22
+L C C80
 U 1 1 58B4A1B4
 P 3700 2350
-F 0 "C22" H 3586 2502 50  0000 R CNN
+F 0 "C80" H 3586 2502 50  0000 R CNN
 F 1 "0.1u" H 3586 2411 50  0000 R CNN
 F 2 "Capacitors_SMD:C_0402" H -2012 -500 50  0001 C CNN
