File: Navi-KiCAD/RF900MHz.sch (KiCad schematic (older format))
At the start: 51 parts, among them J4 0734120110, U1 CC1310F128RGZR, U2 CC1190RGVR, Y3 XRCGB24M000F2P00R0

Commit message: Some BOM consolidation.
Parts:
- D6: value MF-LED-0603-RED -> MF-LED-0603-GREEN
Changed lines of the file:
@@
 P 6200 6750
 F 0 "D6" V 6300 6700 50  0000 R CNN
-F 1 "MF-LED-0603-RED" H 6600 6850 50  0000 R CNN
+F 1 "MF-LED-0603-GREEN" H 6700 6850 50  0000 R CNN
 F 2 "LEDs:LED_0603" H 800 400 50  0001 C CNN
 F 3 "https://s3.amazonaws.com/devpublic1/datasheets/S_110_LTST-C190KRKT-369667.pdf" H 800 400 50  0001 C CNN

Commit message: Completed key routing.
Parts:
- renumbered C88 to C32, C1 to C33, C66 to C34, C2 to C35, C67 to C36, C3 to C37, C4 to C38, C9 to C39, C14 to C40, C15 to C41, C16 to C42, C17 to C43, C18 to C44, C19 to C45, C13 to C46, C20 to C47, C21 to C48, C24 to C49, C25 to C50, C26 to C51, C27 to C52, C28 to C53, C5 to C54, C29 to C55, C6 to C56, C30 to C57, C7 to C58, D6 to D4, J4 to J1, L1 to L10, L2 to L11, L3 to L12, L4 to L13, L8 to L4, L12 to L5, L15 to L6, L13 to L7, L18 to L8, L14 to L9, R35 to R23, R1 to R24, R2 to R25, R3 to R26, R47 to R27, R4 to R28, R9 to R29, U1 to U5, U2 to U6

Commit message: Some more GNC processor routing
Parts:
- L9: value CIH10T22NJNC -> BLM18HE152SN1D
Changed lines of the file:
@@
 EESchema Schematic File Version 2
-LIBS:Navi-rescue
 LIBS:device
 LIBS:rfcom
@@
 LIBS:powerint
 LIBS:onsemi
+LIBS:transistors
+LIBS:ESD_Protection
+LIBS:ftdi
+LIBS:stm32
+LIBS:transf
+LIBS:ttl_ieee
 LIBS:Navi-cache
 EELAYER 26 0
@@
 P 7650 5750
 F 0 "L9" V 7600 5750 50  0000 C CNN
-F 1 "CIH10T22NJNC" V 7725 5750 50  0000 C CNN
+F 1 "BLM18HE152SN1D" V 7725 5750 50  0000 C CNN
 F 2 "Inductors_SMD:L_0603" H 7650 5750 50  0001 C CNN
 F 3 "" H 7650 5750 50  0001 C CNN
@@
 $EndComp
 $Comp
-L +3.3V #PWR?
+L +3.3V #PWR086
 U 1 1 58CDD174
 P 6450 5750
-F 0 "#PWR?" H 6500 5800 50  0001 C CNN
+F 0 "#PWR086" H 6500 5800 50  0001 C CNN
 F 1 "+3.3V" H 6465 5923 50  0000 C CNN
 F 2 "" H -200 1300 50  0001 C CNN
